File: usb.sch (KiCad schematic (older format))
At the start: 21 parts, among them J2 USB_B, J3 Conn_02x03_Odd_Even, J4 Conn_02x02_Odd_Even, U4 ATmega16U2-MU, Y1 Crystal

Commit message: route finish
Connections:
- net at J2.2 (D-), RV2.1: now also RN3.8; no longer RN3.5
- net at J2.3 (D+), RV1.1: now also RN3.5; no longer RN3.8
- net at U4.29 (D+): now also RN3.4; no longer RN3.1
- net at U4.30 (D-): now also RN3.1; no longer RN3.4
Changed lines of the file:
@@
 $Comp
 L Arduino_Uno:RN RN3
-U 1 1 5C164518
+U 4 1 5C164518
 P 2500 4250
 F 0 "RN3" V 2293 4250 50  0000 C CNN
@@
 F 2 "Resistor_SMD:R_Array_Convex_4x0603" V 2430 4250 50  0001 C CNN
 F 3 "~" H 2500 4250 50  0001 C CNN
-	1    2500 4250
+	4    2500 4250
 	0    1    1    0
 $EndComp
 $Comp
 L Arduino_Uno:RN RN3
-U 4 1 5C164596
+U 1 1 5C164596
 P 2950 4350
 F 0 "RN3" V 2743 4350 50  0000 C CNN
@@
 F 2 "Resistor_SMD:R_Array_Convex_4x0603" V 2880 4350 50  0001 C CNN
 F 3 "~" H 2950 4350 50  0001 C CNN
-	4    2950 4350
+	1    2950 4350
 	0    1    1    0
 $EndComp
