File: main.sch (KiCad schematic (older format))
At the start: 22 parts, among them J5 Conn_02x03_Odd_Even, P1 Power, P2 Analog, P3 Digital, P4 Digital, P5 CONN_01X01, P6 CONN_01X01, P7 CONN_01X01, P8 CONN_01X01, SW1 SW_Push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

Commit message: place finish
Parts:
- C10: value C -> 100n
- JP2: footprint Jumper:SolderJumper-2_P1.3mm_Bridged_Pad1.0x1.5mm -> Jumper:SolderJumper-2_P1.3mm_Open_Pad1.0x1.5mm
Changed lines of the file:
@@
 F 0 "JP2" H 6750 4505 50  0000 C CNN
 F 1 "RESET-EN" H 6750 4414 50  0000 C CNN
-F 2 "Jumper:SolderJumper-2_P1.3mm_Bridged_Pad1.0x1.5mm" H 6750 4300 50  0001 C CNN
+F 2 "Jumper:SolderJumper-2_P1.3mm_Open_Pad1.0x1.5mm" H 6750 4300 50  0001 C CNN
 F 3 "~" H 6750 4300 50  0001 C CNN
 	1    6750 4300
@@
 P 7400 4300
 F 0 "C10" V 7652 4300 50  0000 C CNN
-F 1 "C" V 7561 4300 50  0000 C CNN
+F 1 "100n" V 7561 4300 50  0000 C CNN
 F 2 "Capacitor_SMD:C_0603_1608Metric" H 7438 4150 50  0001 C CNN
 F 3 "~" H 7400 4300 50  0001 C CNN

Commit message: route finish
Parts:
- SW1: footprint Button_Switch_SMD:SW_SPST_B3S-1000 -> Button_Switch_SMD:SW_SPST_PTS645
Changed lines of the file:
@@
 F 0 "SW1" V 6204 4998 50  0000 L CNN
 F 1 "SW_Push" V 6295 4998 50  0000 L CNN
-F 2 "Button_Switch_SMD:SW_SPST_B3S-1000" H 6250 5050 50  0001 C CNN
+F 2 "Button_Switch_SMD:SW_SPST_PTS645" H 6250 5050 50  0001 C CNN
 F 3 "" H 6250 5050 50  0001 C CNN
 	1    6250 4850

Commit message: route finish
Parts:
- SW1: value SW_Push -> RESET
Changed lines of the file:
@@
 P 6250 4850
 F 0 "SW1" V 6204 4998 50  0000 L CNN
-F 1 "SW_Push" V 6295 4998 50  0000 L CNN
+F 1 "RESET" V 6295 4998 50  0000 L CNN
 F 2 "Button_Switch_SMD:SW_SPST_PTS645" H 6250 5050 50  0001 C CNN
 F 3 "" H 6250 5050 50  0001 C CNN
